File: PCBs/PCB_Design_Files/Secondary_Board/power_mgmt.kicad_sch (KiCad schematic)
At the start: 0 parts

Commit message: footprints
Parts:
- added BT1: Battery, symbol Device:Battery
- added C1, C2, C3, C4, C5, C6: 4.7u, Capacitor_SMD:C_0603_1608Metric, symbol Device:C
- added D1: D_Zener, symbol Device:D_Zener
- added L1: CIGT201610LH1R0MNE, RES_CIGT201610_SAM, symbol CIGT201610LH1R0MNE:CIGT201610LH1R0MNE
- added Q1: 2N3904, Package_TO_SOT_THT:TO-92_Inline, symbol Transistor_BJT:2N3904
- added R1: 732k, Resistor_SMD:R_0201_0603Metric, symbol Device:R
- added R2: 100k, symbol Device:R
- added R3: 250, Resistor_SMD:R_0201_0603Metric, symbol Device:R
- added R4: 100, Resistor_SMD:R_0201_0603Metric, symbol Device:R
- added R5: 3.96k, Resistor_SMD:R_0201_0603Metric, symbol Device:R
- added R6: 10k, Resistor_SMD:R_0201_0603Metric, symbol Device:R
- added U1: TPS61023DRLR, DRL0006A, symbol TPS61023:TPS61023DRLR
- added U2: TLV9101IDCKR, SC70-5_DCK_TEX, symbol TLV9101:TLV9101IDCKR
Connections:
- new net: R5.1, R6.2, U2.3 (IN-)
- new net: D1.1 (K), R3.2, U2.1 (IN+)
- new net: R1.2, R2.1, U1.1 (FB)
- new net: L1.2, U1.5 (SW)
- new net: R4.1, U2.4 (OUT)
- new net: Q1.2 (B), R4.2
- new net +3.7V: BT1.1 (+), C4.1, C5.1, L1.1, R3.1, U1.2 (EN), U1.3 (VIN)
- new net 3V3: C1.1, C6.1, Q1.1 (E), R5.2
- new net GND: BT1.2 (-), C1.2, C2.2, C3.2, C4.2, C5.2, C6.2, D1.2 (A), R2.2, R6.1, U1.4 (GND), U2.2 (V-)
- new net Vboost: C2.1, C3.1, Q1.3 (C), R1.1, U1.6 (VOUT), U2.5 (V+)
