File: PCBs/PCB_Design_Files/Secondary_Board/power_mgmt.kicad_sch (KiCad schematic)
At the start: 19 parts, among them Q3 MMBT3904, Q4 MMBT3904, U1 TPS61023DRLR, U2 TLV9101IDCKR

Commit message: footprint update
Parts:
- BT1: footprint (none) -> Diode_THT:D_DO-35_SOD27_P7.62mm_Horizontal
- D1: value D_Zener -> 15N122B; footprint (none) -> Diode_THT:D_DO-35_SOD27_P7.62mm_Horizontal
- L1: footprint RES_CIGT201610_SAM -> Project Footprints:RES_CIGT201610_SAM
- Q3, Q4: footprint Package_TO_SOT_SMD:SOT-23 -> Project Footprints:SOT23_FAS
- R1: value 732k -> 73.2k; footprint Resistor_SMD:R_0201_0603Metric -> Project Footprints:0603_resistor
- R10: renamed from R3; footprint Resistor_SMD:R_0201_0603Metric -> Project Footprints:0603_resistor
- R11: renamed from R4; footprint Resistor_SMD:R_0201_0603Metric -> Project Footprints:0603_resistor
- R12: renamed from R5; footprint Resistor_SMD:R_0201_0603Metric -> Project Footprints:0603_resistor
- R13: renamed from R6; footprint Resistor_SMD:R_0201_0603Metric -> Project Footprints:0603_resistor
- R2: value 100k -> 10k; footprint (none) -> Project Footprints:0603_resistor
- U6: renamed from U2; footprint SC70-5_DCK_TEX -> Project Footprints:SC70-5_DCK_TEX
- renumbered C4 to C2, C5 to C3, C2 to C4, C3 to C5, C1 to C6, C6 to C7, U1 to U5
Other:
- note added: "5V"
- note added: "Boost Converter"
- note added: "Low Dropout Regulator"

Commit message: update
Parts:
- BT1: footprint Diode_THT:D_DO-35_SOD27_P7.62mm_Horizontal -> Connector_JST:JST_PH_S2B-PH-K_1x02_P2.00mm_Horizontal
- L1: symbol CIGT201610LH1R0MNE:CIGT201610LH1R0MNE -> Project_Symbols:CIGT201610LH1R0MNE
Connections:
- net Vboost: no longer Q3.3 (C), Q4.3 (C), U6.5 (V+)
- new net +5V: Q3.3 (C), Q4.3 (C), U6.5 (V+)
Changed lines of the file:
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@@
 	(text "Low Dropout Regulator\n"
 		(exclude_from_sim no)
-		(at 225.552 69.85 0)
+		(at 249.936 72.898 0)
 		(effects
 			(font
-				(size 1.27 1.27)
+				(size 1.778 1.778)
+				(thickness 0.3556)
+				(bold yes)
+				(italic yes)
 			)
 		)
@@
 	(text "Boost Converter\n"
 		(exclude_from_sim no)
-		(at 97.282 50.546 0)
+		(at 99.568 54.61 0)
 		(effects
 			(font
-				(size 1.27 1.27)
+				(face "KiCad Font")
+				(size 1.778 1.778)
+				(thickness 0.3556)
+				(bold yes)
+				(italic yes)
 			)
 		)
@@
 			(width 0)
 			(type default)
-		)
-	)
-	(label "Vboost"
-		(at 226.06 78.74 0)
-		(effects
-			(font
-				(size 1.27 1.27)
-			)
-			(justify left bottom)
-		)
-	)
-	(label "Vboost"
-		(at 203.2 93.98 0)
-		(effects
-			(font
-				(size 1.27 1.27)
-			)
-			(justify left bottom)
 		)
 	)
@@
 	)
 	(symbol
+		(lib_id "power:+5V")
+		(at 203.2 93.98 0)
+		(unit 1)
+		(exclude_from_sim no)
+		(in_bom yes)
+		(on_board yes)
+		(dnp no)
+		(fields_autoplaced yes)
+		(property "Reference" "#PWR018"
+			(at 203.2 97.79 0)
+			(effects
+				(font
+					(size 1.27 1.27)
+				)
+				(hide yes)
+			)
+		)
+		(property "Value" "+5V"
+			(at 203.2 88.9 0)
+			(effects
+				(font
+					(size 1.27 1.27)
+				)
+			)
+		)
+		(property "Footprint" ""
+			(at 203.2 93.98 0)
+			(effects
+				(font
+					(size 1.27 1.27)
+				)
+				(hide yes)
+			)
+		)
+		(property "Datasheet" ""
+			(at 203.2 93.98 0)
+			(effects
+				(font
+					(size 1.27 1.27)
+				)
+				(hide yes)
+			)
+		)
+		(property "Description" "Power symbol creates a global label with name \"+5V\""
+			(at 203.2 93.98 0)
+			(effects
+				(font
+					(size 1.27 1.27)
+				)
+				(hide yes)
+			)
+		)
+		(pin "1"
+		)
+		(instances
+			(project ""
+				(path "/2f5986e4-77b2-4f5d-ab91-80ba6228eb8b/3db8306c-5846-4ae5-ba17-fe529edf9e71"
+					(reference "#PWR018")
+					(unit 1)
+				)
+			)
+		)
+	)
+	(symbol
 		(lib_id "power:GND")
 		(at 144.78 111.76 0)
@@
 	)
 	(symbol
-		(lib_id "CIGT201610LH1R0MNE:CIGT201610LH1R0MNE")
+		(lib_id "Project_Symbols:CIGT201610LH1R0MNE")
 		(at 49.53 60.96 0)
 		(unit 1)
@@
 		)
 		(property "Footprint" "Project Footprints:RES_CIGT201610_SAM"
-			(at 49.53 60.96 0)
+			(at 53.34 69.596 0)
 			(effects
 				(font
@@
 		)
 		(property "Datasheet" "CIGT201610LH1R0MNE"
-			(at 49.53 60.96 0)
+			(at 55.88 67.056 0)
 			(effects
 				(font
@@
 	)
 	(symbol
+		(lib_id "power:+5V")
+		(at 226.06 78.74 0)
+		(unit 1)
+		(exclude_from_sim no)
+		(in_bom yes)
+		(on_board yes)
+		(dnp no)
+		(fields_autoplaced yes)
+		(property "Reference" "#PWR019"
+			(at 226.06 82.55 0)
+			(effects
+				(font
+					(size 1.27 1.27)
+				)
+				(hide yes)
+			)
+		)
+		(property "Value" "+5V"
+			(at 226.06 73.66 0)
+			(effects
+				(font
+					(size 1.27 1.27)
+				)
+			)
+		)
+		(property "Footprint" ""
+			(at 226.06 78.74 0)
+			(effects
+				(font
+					(size 1.27 1.27)
+				)
+				(hide yes)
+			)
+		)
+		(property "Datasheet" ""
+			(at 226.06 78.74 0)
+			(effects
+				(font
+					(size 1.27 1.27)
+				)
+				(hide yes)
+			)
+		)
+		(property "Description" "Power symbol creates a global label with name \"+5V\""
+			(at 226.06 78.74 0)
+			(effects
+				(font
+					(size 1.27 1.27)
+				)
+				(hide yes)
+			)
+		)
+		(pin "1"
+		)
+		(instances
+			(project ""
+				(path "/2f5986e4-77b2-4f5d-ab91-80ba6228eb8b/3db8306c-5846-4ae5-ba17-fe529edf9e71"
+					(reference "#PWR019")
+					(unit 1)
+				)
+			)
+		)
+	)
+	(symbol
 		(lib_id "Device:D_Zener")
 		(at 144.78 102.87 270)
@@
 			)
 		)
-		(property "Footprint" "Diode_THT:D_DO-35_SOD27_P7.62mm_Horizontal"
+		(property "Footprint" "Connector_JST:JST_PH_S2B-PH-K_1x02_P2.00mm_Horizontal"
 			(at 27.94 32.766 90)
 			(effects

Commit message: update
Parts:
- BT1: footprint Connector_JST:JST_PH_S2B-PH-K_1x02_P2.00mm_Horizontal -> Diode_THT:D_DO-35_SOD27_P7.62mm_Horizontal
- L1: symbol Project_Symbols:CIGT201610LH1R0MNE -> CIGT201610LH1R0MNE:CIGT201610LH1R0MNE
- U5: footprint DRL0006A -> Project Footprints:DRL0006A
Connections:
- net Vboost is gone; now on net +5V: C4.1, C5.1, R1.1, U5.6 (VOUT)
Other:
- note removed: "5V"
Changed lines of the file:
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@@
 	(text "Low Dropout Regulator\n"
 		(exclude_from_sim no)
-		(at 249.936 72.898 0)
-		(effects
-			(font
-				(size 1.778 1.778)
-				(thickness 0.3556)
-				(bold yes)
-				(italic yes)
-			)
-		)
-	)
-	(text "5V\n"
-		(exclude_from_sim no)
-		(at 134.62 84.836 0)
+		(at 225.552 69.85 0)
 		(effects
 			(font
@@
 	(text "Boost Converter\n"
 		(exclude_from_sim no)
-		(at 99.568 54.61 0)
+		(at 97.282 50.546 0)
 		(effects
 			(font
-				(face "KiCad Font")
-				(size 1.778 1.778)
-				(thickness 0.3556)
-				(bold yes)
-				(italic yes)
+				(size 1.27 1.27)
 			)
 		)
@@
 		)
 	)
-	(label "Vboost"
-		(at 128.27 82.55 0)
-		(fields_autoplaced yes)
+	(label "+5V"
+		(at 226.06 78.74 0)
 		(effects
 			(font
@@
 			(justify left bottom)
 		)
-		(property "Netclass" ""
-			(at 128.27 83.82 0)
-			(effects
-				(font
-					(size 1.27 1.27)
-					(italic yes)
-				)
-				(justify left)
-			)
+	)
+	(label "+5V"
+		(at 203.2 93.98 0)
+		(effects
+			(font
+				(size 1.27 1.27)
+			)
+			(justify left bottom)
 		)
 	)
@@
 		)
 	)
+	(hierarchical_label "+5V"
+		(shape input)
+		(at 128.27 82.55 0)
+		(effects
+			(font
+				(size 1.27 1.27)
+			)
+			(justify left)
+		)
+	)
 	(symbol
 		(lib_id "Device:R")
@@
 	)
 	(symbol
-		(lib_id "power:+5V")
-		(at 203.2 93.98 0)
-		(unit 1)
-		(exclude_from_sim no)
-		(in_bom yes)
-		(on_board yes)
-		(dnp no)
-		(fields_autoplaced yes)
-		(property "Reference" "#PWR018"
-			(at 203.2 97.79 0)
-			(effects
-				(font
-					(size 1.27 1.27)
-				)
-				(hide yes)
-			)
-		)
-		(property "Value" "+5V"
-			(at 203.2 88.9 0)
-			(effects
-				(font
-					(size 1.27 1.27)
-				)
-			)
-		)
-		(property "Footprint" ""
-			(at 203.2 93.98 0)
-			(effects
-				(font
-					(size 1.27 1.27)
-				)
-				(hide yes)
-			)
-		)
-		(property "Datasheet" ""
-			(at 203.2 93.98 0)
-			(effects
-				(font
-					(size 1.27 1.27)
-				)
-				(hide yes)
-			)
-		)
-		(property "Description" "Power symbol creates a global label with name \"+5V\""
-			(at 203.2 93.98 0)
-			(effects
-				(font
-					(size 1.27 1.27)
-				)
-				(hide yes)
-			)
-		)
-		(pin "1"
-		)
-		(instances
-			(project ""
-				(path "/2f5986e4-77b2-4f5d-ab91-80ba6228eb8b/3db8306c-5846-4ae5-ba17-fe529edf9e71"
-					(reference "#PWR018")
-					(unit 1)
-				)
-			)
-		)
-	)
-	(symbol
 		(lib_id "power:GND")
 		(at 144.78 111.76 0)
@@
 	)
 	(symbol
-		(lib_id "Project_Symbols:CIGT201610LH1R0MNE")
+		(lib_id "CIGT201610LH1R0MNE:CIGT201610LH1R0MNE")
 		(at 49.53 60.96 0)
 		(unit 1)
@@
 		)
 		(property "Footprint" "Project Footprints:RES_CIGT201610_SAM"
-			(at 53.34 69.596 0)
+			(at 49.53 60.96 0)
 			(effects
 				(font
@@
 		)
 		(property "Datasheet" "CIGT201610LH1R0MNE"
-			(at 55.88 67.056 0)
+			(at 49.53 60.96 0)
 			(effects
 				(font
@@
 			)
 		)
-		(property "Footprint" "DRL0006A"
+		(property "Footprint" "Project Footprints:DRL0006A"
 			(at 55.88 82.55 0)
 			(effects
@@
 	)
 	(symbol
-		(lib_id "power:+5V")
-		(at 226.06 78.74 0)
-		(unit 1)
-		(exclude_from_sim no)
-		(in_bom yes)
-		(on_board yes)
-		(dnp no)
-		(fields_autoplaced yes)
-		(property "Reference" "#PWR019"
-			(at 226.06 82.55 0)
-			(effects
-				(font
-					(size 1.27 1.27)
-				)
-				(hide yes)
-			)
-		)
-		(property "Value" "+5V"
-			(at 226.06 73.66 0)
-			(effects
-				(font
-					(size 1.27 1.27)
-				)
-			)
-		)
-		(property "Footprint" ""
-			(at 226.06 78.74 0)
-			(effects
-				(font
-					(size 1.27 1.27)
-				)
-				(hide yes)
-			)
-		)
-		(property "Datasheet" ""
-			(at 226.06 78.74 0)
-			(effects
-				(font
-					(size 1.27 1.27)
-				)
-				(hide yes)
-			)
-		)
-		(property "Description" "Power symbol creates a global label with name \"+5V\""
-			(at 226.06 78.74 0)
-			(effects
-				(font
-					(size 1.27 1.27)
-				)
-				(hide yes)
-			)
-		)
-		(pin "1"
-		)
-		(instances
-			(project ""
-				(path "/2f5986e4-77b2-4f5d-ab91-80ba6228eb8b/3db8306c-5846-4ae5-ba17-fe529edf9e71"
-					(reference "#PWR019")
-					(unit 1)
-				)
-			)
-		)
-	)
-	(symbol
 		(lib_id "Device:D_Zener")
 		(at 144.78 102.87 270)
@@
 			)
 		)
-		(property "Footprint" "Connector_JST:JST_PH_S2B-PH-K_1x02_P2.00mm_Horizontal"
+		(property "Footprint" "Diode_THT:D_DO-35_SOD27_P7.62mm_Horizontal"
 			(at 27.94 32.766 90)
 			(effects

Commit message: updte
Parts:
- removed U5: TPS61023DRLR, Project Footprints:DRL0006A, symbol TPS61023:TPS61023DRLR
- added U5: TPS61023DRLR, Project Footprints:DRL0006A, symbol Project_Symbols:TPS61023DRLR
- BT1: footprint Diode_THT:D_DO-35_SOD27_P7.62mm_Horizontal -> Connector_JST:JST_PH_S2B-PH-K_1x02_P2.00mm_Horizontal
Connections:
- net +3.7V: now also U5.2 (EN), U5.3 (VIN)
- net +5V: now also U5.6 (VOUT)
- net GND: now also U5.4 (GND)
- net at R1.2, R2.1: now also U5.1 (FB)
- net at L1.2: now also U5.5 (SW)
Changed lines of the file:
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@@
+	)
+	(junction
+		(at 36.83 87.63)
+		(diameter 0)
+		(color 0 0 0 0)
 	)
 	(junction
@@
 	)
 	(junction
-		(at 36.83 87.63)
-		(diameter 0)
-		(color 0 0 0 0)
-	)
-	(junction
 		(at 113.03 82.55)
 		(diameter 0)
@@
 	)
 	(junction
-		(at 38.1 77.47)
-		(diameter 0)
-		(color 0 0 0 0)
-	)
-	(junction
 		(at 91.44 82.55)
 		(diameter 0)
@@
 	)
 	(junction
+		(at 36.83 77.47)
+		(diameter 0)
+		(color 0 0 0 0)
+	)
+	(junction
 		(at 91.44 110.49)
 		(diameter 0)
@@
 	(wire
 		(pts
+			(xy 31.75 87.63) (xy 36.83 87.63)
+		)
+		(stroke
+			(width 0)
+			(type default)
+		)
+	)
+	(wire
+		(pts
 			(xy 157.48 95.25) (xy 144.78 95.25)
 		)
@@
 	(wire
 		(pts
-			(xy 38.1 77.47) (xy 38.1 82.55)
-		)
-		(stroke
-			(width 0)
-			(type default)
-		)
-	)
-	(wire
-		(pts
 			(xy 91.44 92.71) (xy 91.44 93.98)
 		)
@@
 	(wire
 		(pts
-			(xy 38.1 87.63) (xy 36.83 87.63)
-		)
-		(stroke
-			(width 0)
-			(type default)
-		)
-	)
-	(wire
-		(pts
 			(xy 25.4 85.09) (xy 25.4 88.9)
 		)
@@
 	(wire
 		(pts
+			(xy 36.83 77.47) (xy 38.1 77.47)
+		)
+		(stroke
+			(width 0)
+			(type default)
+		)
+	)
+	(wire
+		(pts
 			(xy 144.78 95.25) (xy 144.78 99.06)
 		)
@@
 	(wire
 		(pts
+			(xy 29.21 77.47) (xy 36.83 77.47)
+		)
+		(stroke
+			(width 0)
+			(type default)
+		)
+	)
+	(wire
+		(pts
 			(xy 229.87 99.06) (xy 229.87 80.01)
 		)
@@
 	(wire
 		(pts
-			(xy 36.83 87.63) (xy 31.75 87.63)
-		)
-		(stroke
-			(width 0)
-			(type default)
-		)
-	)
-	(wire
-		(pts
 			(xy 91.44 93.98) (xy 91.44 96.52)
 		)
@@
 	(wire
 		(pts
+			(xy 38.1 82.55) (xy 36.83 82.55)
+		)
+		(stroke
+			(width 0)
+			(type default)
+		)
+	)
+	(wire
+		(pts
 			(xy 49.53 60.96) (xy 17.78 60.96)
 		)
@@
 	(wire
 		(pts
-			(xy 29.21 77.47) (xy 38.1 77.47)
+			(xy 36.83 87.63) (xy 38.1 87.63)
 		)
 		(stroke
@@
 		(pts
 			(xy 254 134.62) (xy 254 130.81)
+		)
+		(stroke
+			(width 0)
+			(type default)
+		)
+	)
+	(wire
+		(pts
+			(xy 36.83 77.47) (xy 36.83 82.55)
 		)
 		(stroke
@@
 	)
 	(symbol
-		(lib_id "TPS61023:TPS61023DRLR")
-		(at 55.88 82.55 0)
-		(unit 1)
-		(exclude_from_sim no)
-		(in_bom yes)
-		(on_board no)
-		(dnp no)
-		(fields_autoplaced yes)
-		(property "Reference" "U5"
-			(at 55.88 67.31 0)
-			(effects
-				(font
-					(size 1.524 1.524)
-				)
-			)
-		)
-		(property "Value" "TPS61023DRLR"
-			(at 55.88 69.85 0)
-			(effects
-				(font
-					(size 1.524 1.524)
-				)
-			)
-		)
-		(property "Footprint" "Project Footprints:DRL0006A"
-			(at 55.88 82.55 0)
-			(effects
-				(font
-					(size 1.27 1.27)
-					(italic yes)
-				)
-				(hide yes)
-			)
-		)
-		(property "Datasheet" "https://www.ti.com/lit/gpn/tps61023"
-			(at 55.88 82.55 0)
-			(effects
-				(font
-					(size 1.27 1.27)
-					(italic yes)
-				)
-				(hide yes)
-			)
-		)
-		(property "Description" ""
-			(at 55.88 82.55 0)
-			(effects
-				(font
-					(size 1.27 1.27)
-				)
-				(hide yes)
-			)
-		)
-		(pin "1"
-		)
-		(pin "6"
-		)
-		(pin "3"
-		)
-		(pin "4"
-		)
-		(pin "5"
-		)
-		(pin "2"
-		)
-		(instances
-			(project "Secondary_Board"
-				(path "/2f5986e4-77b2-4f5d-ab91-80ba6228eb8b/3db8306c-5846-4ae5-ba17-fe529edf9e71"
-					(reference "U5")
-					(unit 1)
-				)
-			)
-			(project "power_mgmt"
-				(path "/c7abdc65-9966-45f8-babc-768b62a50249"
-					(reference "U1")
-					(unit 1)
-				)
-			)
-		)
-	)
-	(symbol
 		(lib_id "power:PWR_FLAG")
 		(at 36.83 26.67 0)
@@
 	)
 	(symbol
+		(lib_id "Project_Symbols:TPS61023DRLR")
+		(at 55.88 82.55 0)
+		(unit 1)
+		(exclude_from_sim no)
+		(in_bom yes)
+		(on_board yes)
+		(dnp no)
+		(fields_autoplaced yes)
+		(property "Reference" "U5"
+			(at 55.88 67.31 0)
+			(effects
+				(font
+					(size 1.524 1.524)
+				)
+			)
+		)
+		(property "Value" "TPS61023DRLR"
+			(at 55.88 69.85 0)
+			(effects
+				(font
+					(size 1.524 1.524)
+				)
+			)
+		)
+		(property "Footprint" "Project Footprints:DRL0006A"
+			(at 55.372 95.25 0)
+			(effects
+				(font
+					(size 1.27 1.27)
+					(italic yes)
+				)
+				(hide yes)
+			)
+		)
+		(property "Datasheet" "https://www.ti.com/lit/gpn/tps61023"
+			(at 57.15 93.472 0)
+			(effects
+				(font
+					(size 1.27 1.27)
+					(italic yes)
+				)
+				(hide yes)
+			)
+		)
+		(property "Description" ""
+			(at 55.88 82.55 0)
+			(effects
+				(font
+					(size 1.27 1.27)
+				)
+				(hide yes)
+			)
+		)
+		(pin "5"
+		)
+		(pin "6"
+		)
+		(pin "1"
+		)
+		(pin "3"
+		)
+		(pin "2"
+		)
+		(pin "4"
+		)
+		(instances
+			(project ""
+				(path "/2f5986e4-77b2-4f5d-ab91-80ba6228eb8b/3db8306c-5846-4ae5-ba17-fe529edf9e71"
+					(reference "U5")
+					(unit 1)
+				)
+			)
+		)
+	)
+	(symbol
 		(lib_id "Device:C")
 		(at 21.59 81.28 0)
@@
 			)
 		)
-		(property "Footprint" "Diode_THT:D_DO-35_SOD27_P7.62mm_Horizontal"
+		(property "Footprint" "Connector_JST:JST_PH_S2B-PH-K_1x02_P2.00mm_Horizontal"
 			(at 27.94 32.766 90)
 			(effects

Commit message: boost to PCB
Parts:
- removed L1: CIGT201610LH1R0MNE, Project Footprints:RES_CIGT201610_SAM, symbol CIGT201610LH1R0MNE:CIGT201610LH1R0MNE
- added L1: XEL4030-102MEB, Project Footprints:IND_XEL4030_3.1_COC, symbol Project_Symbols:XEL4030-102MEB
- C4, C5: value 4.7u -> 22u
- R1: value 73.2k -> 732k
- R2: value 10k -> 100k
Connections:
- net +3.7V: now also L1.1
- net Vfb: now reaches R1.2, R2.1, U5.1 (FB)
- net at U5.5 (SW): now also L1.2
Changed lines of the file:
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@@
+	(wire
+		(pts
+			(xy 46.99 60.96) (xy 17.78 60.96)
+		)
+		(stroke
+			(width 0)
+			(type default)
+		)
+	)
 	(wire
 		(pts
@@
 		(pts
 			(xy 38.1 82.55) (xy 36.83 82.55)
-		)
-		(stroke
-			(width 0)
-			(type default)
-		)
-	)
-	(wire
-		(pts
-			(xy 49.53 60.96) (xy 17.78 60.96)
 		)
 		(stroke
@@
 	(label "+5V"
 		(at 226.06 78.74 0)
+		(effects
+			(font
+				(size 1.27 1.27)
+			)
+			(justify left bottom)
+		)
+	)
+	(label "Vfb"
+		(at 91.44 93.98 0)
 		(effects
 			(font
@@
 	)
 	(symbol
+		(lib_id "Project_Symbols:XEL4030-102MEB")
+		(at 62.23 60.96 0)
+		(mirror y)
+		(unit 1)
+		(exclude_from_sim no)
+		(in_bom yes)
+		(on_board yes)
+		(dnp no)
+		(property "Reference" "L1"
+			(at 54.61 53.34 0)
+			(effects
+				(font
+					(size 1.524 1.524)
+				)
+			)
+		)
+		(property "Value" "XEL4030-102MEB"
+			(at 54.61 55.88 0)
+			(effects
+				(font
+					(size 1.524 1.524)
+				)
+			)
+		)
+		(property "Footprint" "Project Footprints:IND_XEL4030_3.1_COC"
+			(at 62.23 60.96 0)
+			(effects
+				(font
+					(size 1.27 1.27)
+					(italic yes)
+				)
+				(hide yes)
+			)
+		)
+		(property "Datasheet" "XEL4030-102MEB"
+			(at 62.23 60.96 0)
+			(effects
+				(font
+					(size 1.27 1.27)
+					(italic yes)
+				)
+				(hide yes)
+			)
+		)
+		(property "Description" ""
+			(at 62.23 60.96 0)
+			(effects
+				(font
+					(size 1.27 1.27)
+				)
+				(hide yes)
+			)
+		)
+		(pin "1"
+		)
+		(pin "2"
+		)
+		(instances
+			(project ""
+				(path "/2f5986e4-77b2-4f5d-ab91-80ba6228eb8b/3db8306c-5846-4ae5-ba17-fe529edf9e71"
+					(reference "L1")
+					(unit 1)
+				)
+			)
+		)
+	)
+	(symbol
 		(lib_id "power:PWR_FLAG")
 		(at 36.83 39.37 0)
@@
 			)
 		)
-		(property "Value" "73.2k"
+		(property "Value" "732k"
 			(at 93.98 90.1699 0)
 			(effects
@@
 			)
 		)
-		(property "Value" "10k"
+		(property "Value" "100k"
 			(at 93.98 101.5999 0)
 			(effects
@@
 			)
 		)
-		(property "Value" "4.7u"
+		(property "Value" "22u"
 			(at 127 87.6299 0)
 			(effects
@@
 	)
 	(symbol
-		(lib_id "CIGT201610LH1R0MNE:CIGT201610LH1R0MNE")
-		(at 49.53 60.96 0)
-		(unit 1)
-		(exclude_from_sim no)
-		(in_bom yes)
-		(on_board yes)
-		(dnp no)
-		(fields_autoplaced yes)
-		(property "Reference" "L1"
-			(at 55.88 54.61 0)
-			(effects
-				(font
-					(size 1.524 1.524)
-				)
-			)
-		)
-		(property "Value" "CIGT201610LH1R0MNE"
-			(at 55.88 57.15 0)
-			(effects
-				(font
-					(size 1.524 1.524)
-				)
-			)
-		)
-		(property "Footprint" "Project Footprints:RES_CIGT201610_SAM"
-			(at 49.53 60.96 0)
-			(effects
-				(font
-					(size 1.27 1.27)
-					(italic yes)
-				)
-				(hide yes)
-			)
-		)
-		(property "Datasheet" "CIGT201610LH1R0MNE"
-			(at 49.53 60.96 0)
-			(effects
-				(font
-					(size 1.27 1.27)
-					(italic yes)
-				)
-				(hide yes)
-			)
-		)
-		(property "Description" ""
-			(at 49.53 60.96 0)
-			(effects
-				(font
-					(size 1.27 1.27)
-				)
-				(hide yes)
-			)
-		)
-		(pin "1"
-		)
-		(pin "2"
-		)
-		(instances
-			(project "Secondary_Board"
-				(path "/2f5986e4-77b2-4f5d-ab91-80ba6228eb8b/3db8306c-5846-4ae5-ba17-fe529edf9e71"
-					(reference "L1")
-					(unit 1)
-				)
-			)
-			(project "power_mgmt"
-				(path "/c7abdc65-9966-45f8-babc-768b62a50249"
-					(reference "L1")
-					(unit 1)
-				)
-			)
-		)
-	)
-	(symbol
 		(lib_id "power:GND")
 		(at 25.4 88.9 0)
@@
 			)
 		)
-		(property "Value" "4.7u"
+		(property "Value" "22u"
 			(at 116.84 87.6299 0)
 			(effects

Commit message: updated ptat_bandgap schematic and layout. Fixed +3v3 and +5V flags
Connections:
- net 3V3 renamed +3V3
