File: PCBs/PCB_Design_Files/Secondary_Board/LED_Driver.kicad_sch (KiCad schematic)
At the start: 14 parts, among them Q1 MMBT3904, Q2 MMBT3904, Q5 2N7002, Q6 BSS84, Q7 2N7002, Q8 BSS84, U8 OPA333AIDCKR

Commit message: final checks
Changed lines of the file:
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@@
 	(wire
 		(pts
-			(xy 191.77 121.92) (xy 195.58 121.92)
+			(xy 191.77 121.92) (xy 208.28 121.92)
 		)
 		(stroke
@@
 	(hierarchical_label "V_bandgap"
 		(shape input)
-		(at 195.58 121.92 0)
-		(effects
-			(font
+		(at 208.28 121.92 0)
+		(effects
+			(font

Commit message: added pull up to bg led driver
Parts:
- added R20: 10k, Resistor_SMD:R_0603_1608Metric_Pad0.98x0.95mm_HandSolder, symbol Device:R
Connections:
- net V_bandgap: now also R20.1; no longer Q7.3, U8.1 (+IN)
- new net: Q7.3, R20.2, U8.1 (+IN)
Changed lines of the file:
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@@
 	(wire
 		(pts
-			(xy 191.77 121.92) (xy 208.28 121.92)
+			(xy 191.77 121.92) (xy 195.58 121.92)
 		)
 		(stroke
@@
 		(pts
 			(xy 176.53 80.01) (xy 176.53 102.87)
+		)
+		(stroke
+			(width 0)
+			(type default)
+		)
+	)
+	(wire
+		(pts
+			(xy 203.2 121.92) (xy 208.28 121.92)
 		)
 		(stroke
@@
 					(unit 1)
 				)
+			)
+		)
+	)
+	(symbol
+		(lib_id "Device:R")
+		(at 199.39 121.92 270)
+		(unit 1)
+		(exclude_from_sim no)
+		(in_bom yes)
+		(on_board yes)
+		(dnp no)
+		(fields_autoplaced yes)
+		(property "Reference" "R20"
+			(at 199.39 115.57 90)
+			(effects
+				(font
+					(size 1.27 1.27)
+				)
+			)
+		)
+		(property "Value" "10k"
+			(at 199.39 118.11 90)
+			(effects
+				(font
+					(size 1.27 1.27)
+				)
+			)
+		)
+		(property "Footprint" "Resistor_SMD:R_0603_1608Metric_Pad0.98x0.95mm_HandSolder"
+			(at 199.39 120.142 90)
+			(effects
+				(font
+					(size 1.27 1.27)
+				)
+				(hide yes)
+			)
+		)
+		(property "Datasheet" "~"
+			(at 199.39 121.92 0)
+			(effects
+				(font
+					(size 1.27 1.27)
+				)
+				(hide yes)
+			)
+		)
+		(property "Description" "Resistor"
+			(at 199.39 121.92 0)
+			(effects
+				(font
+					(size 1.27 1.27)
+				)
+				(hide yes)
+			)
+		)
+		(pin "2"
+		)
+		(pin "1"
+		)
+		(instances
+			(project "Secondary_Board"
+				(path "/2f5986e4-77b2-4f5d-ab91-80ba6228eb8b/16ecf950-1853-427b-9137-65792483b2a5"
+					(reference "R20")
+					(unit 1)
+				)
